Commit message: map created for navigation. amcl parameters to be tuned

File: catkin_ws/src/my_robot/urdf/my_robot.xacro (robot description, xacro)
@@ -33,5 +33,5 @@
     </visual>
    <collision name="front_caster_collision">
-      <origin xyz="0.1 0 -0.05" rpy="0 0 0" />
+      <origin xyz="0.15 0 -0.05" rpy="0 0 0" />
       <geometry>
         <sphere radius="0.0499" />
@@ -39,5 +39,17 @@
     </collision>
    <visual name="front_caster_visual">
-      <origin xyz="0.1 0 -0.05" rpy="0 0 0" />
+      <origin xyz="0.15 0 -0.05" rpy="0 0 0" />
+      <geometry>
+        <sphere radius="0.0499" />
+      </geometry>
+    </visual>
+   <collision name="back_caster_collision">
+      <origin xyz="-0.15 0 -0.05" rpy="0 0 0" />
+      <geometry>
+        <sphere radius="0.0499" />
+      </geometry>
+    </collision>
+   <visual name="back_caster_visual">
+      <origin xyz="-0.15 0 -0.05" rpy="0 0 0" />
       <geometry>
         <sphere radius="0.0499" />
